File: contactlessReader_licensed.kicad_pcb (KiCad board)
At the start: 2 copper layers, 85.7 x 61.2 mm, 41 parts, among them J1 Conn_01x04_Male, J2 Conn_01x08_Male

Commit message: rev. 2.3.1
Parts:
- removed CRX1: CRX, TestPoint:TestPoint_Pad_1.0x1.0mm
- removed CRX2: CRX2, TestPoint:TestPoint_Pad_1.0x1.0mm
- removed CTX1: CTX, TestPoint:TestPoint_Pad_1.0x1.0mm
- removed CTX2: CTX2, TestPoint:TestPoint_Pad_1.0x1.0mm
- added G***: LOGO, AeonLabs:pcbWay Logo Collab, F.Cu at (162.4, 137.9)
- added RX1: RX1, TestPoint:TestPoint_Pad_Bridge_1.0x1.0mm, B.Cu at (121.0, 131.0)
- added TX1: TX1, TestPoint:TestPoint_Pad_Bridge_1.0x1.0mm, B.Cu at (121.0, 133.4)
- ENR1, LEDR1, LEDR2, LEDR3: footprint Resistor_SMD:R_1206_3216Metric -> Resistor_SMD:R_1206_3216Metric_Pad1.30x1.75mm_HandSolder
- ESPC1, ESPC2, ESP_EN_C1, HXC1, HXC2, HXC3, HXC4: footprint Capacitor_SMD:C_1206_3216Metric -> Capacitor_SMD:C_1206_3216Metric_Pad1.33x1.80mm_HandSolder
- Fuse1: footprint Fuse:Fuse_1206_3216Metric -> Fuse:Fuse_1206_3216Metric_Pad1.42x1.75mm_HandSolder
- HX4002B1, HX4002B2: footprint Package_SO:SOT95P280X125-6N -> AeonLabs:HX4002 SOT95 P280X125-6N
- PWC1: footprint Capacitor_SMD:C_True_1206_3216Metric -> Capacitor_SMD:C_1206_3216Metric_Pad1.33x1.80mm_HandSolder
- moved RGBLED1 3.20 mm to (103.6, 101.7)
- moved G*** 1.26 mm to (129.5, 138.5)
- moved G*** 0.38 mm to (144.2, 133.0)
- moved HX4002B1 0.27 mm to (115.4, 117.2)
- moved ESP_EN_C1 0.16 mm to (182.7, 117.4)
- moved HX4002B2 0.13 mm to (115.2, 113.4)
- moved BUZZER1 0.06 mm to (116.8, 88.9)
Routing:
- net /GND: track 228.8 -> 232.7 mm
- net Net-(LEDR3-Pad1): track 6.26 -> 7.91 mm
- net Net-(LEDR1-Pad1): track 7.58 -> 6.03 mm
- net /IO13: track 66.8 -> 67.3 mm
Other:
- board text added: "86x62mm board rev. 2.3.1"
- board text added: "Contact AeonLabs for a Commercial License"
- board text added: "WIFI BLE RFID NFC contactless"
- board text removed: "86x62mm"
- board text removed: "WIFI BLE RFID NFC contactless board rev. 2.3"
