File: contactlessReader_licensed.kicad_sch (KiCad schematic)
At the start: 38 parts, among them J1 Conn_01x04_Male, J2 Conn_01x08_Male

Commit message: rev. 2.3.1
Parts:
- removed CRX1: CRX, TestPoint:TestPoint_Pad_1.0x1.0mm, symbol Connector:TestPoint
- removed CRX2: CRX2, TestPoint:TestPoint_Pad_1.0x1.0mm, symbol Connector:TestPoint
- removed CTX1: CTX, TestPoint:TestPoint_Pad_1.0x1.0mm, symbol Connector:TestPoint
- removed CTX2: CTX2, TestPoint:TestPoint_Pad_1.0x1.0mm, symbol Connector:TestPoint
- added RX1: RX1, TestPoint:TestPoint_Pad_Bridge_1.0x1.0mm, symbol Connector:TestPoint_2Pole
- added TX1: TX1, TestPoint:TestPoint_Pad_Bridge_1.0x1.0mm, symbol Connector:TestPoint_2Pole
- ENR1, LEDR1, LEDR2, LEDR3: footprint Resistor_SMD:R_1206_3216Metric -> Resistor_SMD:R_1206_3216Metric_Pad1.30x1.75mm_HandSolder
- ESPC1, ESPC2, ESP_EN_C1, HXC1, HXC2, HXC3, HXC4: footprint Capacitor_SMD:C_1206_3216Metric -> Capacitor_SMD:C_1206_3216Metric_Pad1.33x1.80mm_HandSolder
- Fuse1: footprint Fuse:Fuse_1206_3216Metric -> Fuse:Fuse_1206_3216Metric_Pad1.42x1.75mm_HandSolder
- HX4002B1, HX4002B2: footprint Package_SO:SOT95P280X125-6N -> AeonLabs:HX4002 SOT95 P280X125-6N
- PWC1: footprint Capacitor_SMD:C_True_1206_3216Metric -> Capacitor_SMD:C_1206_3216Metric_Pad1.33x1.80mm_HandSolder
Connections:
- net IO01TX: now also RX1.2
- net IO03RX: now also TX1.2
- net RX_IN: now also RX1.1
- net TX_IN: now also TX1.1
Other:
- moved on the sheet: BAT+1, BAT-1, BUZZER1, ENR1, ESP32-WROOM32, ESPC1, ESPC2, ESP_EN_C1, Fuse1, H1, H2, H3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
